File: motor.kicad_sch (KiCad schematic)
At the start: 2 parts

Commit message: 回路設計済
Parts:
- J2: renamed from J?; footprint (none) -> Connector_PinSocket_1.27mm:PinSocket_1x02_P1.27mm_Vertical
- U2: renamed from U?; footprint (none) -> omni:DRV8835
Changed lines of the file:
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@@
   (symbol (lib_id "Connector_Generic:Conn_01x02") (at 157.48 80.01 0) (unit 1)
     (in_bom yes) (on_board yes) (fields_autoplaced)
-    (property "Reference" "J?" (id 0) (at 160.02 80.0099 0)
+    (property "Reference" "J2" (id 0) (at 160.02 80.0099 0)
       (effects (font (size 1.27 1.27)) (justify left))
     )
@@
       (effects (font (size 1.27 1.27)) (justify left))
     )
-    (property "Footprint" "" (id 2) (at 157.48 80.01 0)
+    (property "Footprint" "Connector_PinSocket_1.27mm:PinSocket_1x02_P1.27mm_Vertical" (id 2) (at 157.48 80.01 0)
       (effects (font (size 1.27 1.27)) hide)
     )
@@
   (symbol (lib_id "power:+3.3V") (at 132.08 72.39 0) (unit 1)
     (in_bom yes) (on_board yes) (fields_autoplaced)
-    (property "Reference" "#PWR?" (id 0) (at 132.08 76.2 0)
+    (property "Reference" "#PWR07" (id 0) (at 132.08 76.2 0)
       (effects (font (size 1.27 1.27)) hide)
     )
@@
   (symbol (lib_id "My_Device:DRV8835") (at 133.35 66.04 0) (unit 1)
     (in_bom yes) (on_board yes) (fields_autoplaced)
-    (property "Reference" "U?" (id 0) (at 137.9094 72.39 0)
+    (property "Reference" "U2" (id 0) (at 137.9094 72.39 0)
       (effects (font (size 1.27 1.27)) (justify left))
     )
@@
       (effects (font (size 1.27 1.27)) (justify left))
     )
-    (property "Footprint" "" (id 2) (at 133.35 66.04 0)
+    (property "Footprint" "omni:DRV8835" (id 2) (at 133.35 66.04 0)
       (effects (font (size 1.27 1.27)) hide)
     )
@@
   (symbol (lib_id "power:GND") (at 135.89 101.6 0) (unit 1)
     (in_bom yes) (on_board yes) (fields_autoplaced)
-    (property "Reference" "#PWR?" (id 0) (at 135.89 107.95 0)
+    (property "Reference" "#PWR010" (id 0) (at 135.89 107.95 0)
       (effects (font (size 1.27 1.27)) hide)
     )
@@
   (symbol (lib_id "power:GND") (at 132.08 101.6 0) (unit 1)
     (in_bom yes) (on_board yes) (fields_autoplaced)
-    (property "Reference" "#PWR?" (id 0) (at 132.08 107.95 0)
+    (property "Reference" "#PWR08" (id 0) (at 132.08 107.95 0)
       (effects (font (size 1.27 1.27)) hide)
     )
@@
   (symbol (lib_id "power:GND") (at 118.11 96.52 0) (unit 1)
     (in_bom yes) (on_board yes) (fields_autoplaced)
-    (property "Reference" "#PWR?" (id 0) (at 118.11 102.87 0)
+    (property "Reference" "#PWR06" (id 0) (at 118.11 102.87 0)
       (effects (font (size 1.27 1.27)) hide)
     )
@@
   (symbol (lib_id "power:+BATT") (at 135.89 69.85 0) (unit 1)
     (in_bom yes) (on_board yes) (fields_autoplaced)
-    (property "Reference" "#PWR?" (id 0) (at 135.89 73.66 0)
+    (property "Reference" "#PWR09" (id 0) (at 135.89 73.66 0)
       (effects (font (size 1.27 1.27)) hide)
     )
