File: controller.kicad_sch (KiCad schematic)
At the start: 10 parts

Commit message: 回路設計済
Parts:
- added C22: 1u, Capacitor_SMD:C_0603_1608Metric_Pad1.08x0.95mm_HandSolder, symbol Device:C_Small
- C14, C15, C16, C17, C18, C19, C20: renamed from C?; footprint (none) -> Capacitor_SMD:C_0603_1608Metric_Pad1.08x0.95mm_HandSolder
- C21: renamed from C?; value 0.1u -> 0.01u; footprint (none) -> Capacitor_SMD:C_0603_1608Metric_Pad1.08x0.95mm_HandSolder
- R12: renamed from R?; footprint (none) -> Resistor_SMD:R_0805_2012Metric_Pad1.20x1.40mm_HandSolder
- gave numbers to parts that had none: 1
Connections:
- net +3.3VADC: now also C22.1
- net GND: now also C22.2
Other:
- moved on the sheet: R12

Commit message: 部品配置完了
Parts:
- removed U13: STM32F446RE, Package_QFP:LQFP-64_10x10mm_P0.5mm, symbol My_Device:STM32F446RE
- added J15, J17: Conn_01x08_Female, Connector_JST:JST_SH_SM08B-SRSS-TB_1x08-1MP_P1.00mm_Horizontal, symbol Connector:Conn_01x08_Female
- added J16, J18: Conn_01x11_Female, Connector_JST:JST_SH_SM11B-SRSS-TB_1x11-1MP_P1.00mm_Horizontal, symbol Connector:Conn_01x11_Female
- added U12: STM32F446RE, Package_QFP:LQFP-64_10x10mm_P0.5mm, symbol bldc_lib:STM32F446RE
Connections:
- net +3.3VADC is gone; now on net +3.3V: C21.1, C22.1
- net +3.3V: now also J16.10 (Pin_10), U12.1 (VBAT), U12.13 (VDDA), U12.19 (VDD), U12.32 (VDD), U12.48 (VDD), U12.64 (VDD)
- net ADC_BAT: now also J18.4 (Pin_4)
- net BOOT0: now also U12.60 (BOOT0)
- net BUTTON_OUTPUT: now also U12.28 (PB2)
- net BUZZER_INPUT: now also U12.16 (PA2)
- net GND: now also J16.11 (Pin_11), U12.12 (VSSA), U12.18 (VSS), U12.31 (VSS), U12.63 (VSS)
- net LED1: now also U12.36 (PB15)
- net LED2: now also U12.35 (PB14)
- net LED3: now also U12.34 (PB13)
- net LED4: now also U12.33 (PB12)
- net MOTOR1_IN1: now also J18.8 (Pin_8)
- net MOTOR1_IN2: now also J18.9 (Pin_9)
- net MOTOR2_IN1: now also J17.8 (Pin_8)
- net MOTOR2_IN2: now also J17.7 (Pin_7)
- net MOTOR3_IN1: now also J18.10 (Pin_10)
- net MOTOR3_IN2: now also J18.11 (Pin_11)
- net MOTOR4_IN1: now also J18.3 (Pin_3)
- net MOTOR4_IN2: now also J18.7 (Pin_7)
- net MOTOR5_IN1: now also J17.1 (Pin_1)
- net MOTOR5_IN2: now also J17.2 (Pin_2)
- net MOTOR6_IN1: now also J17.3 (Pin_3)
- net MOTOR6_IN2: now also J17.4 (Pin_4)
- net MOTOR7_IN1: now also J17.5 (Pin_5)
- net MOTOR7_IN2: now also J17.6 (Pin_6)
- net MOTOR8_IN1: now also J18.5 (Pin_5)
- net MOTOR8_IN2: now also J18.6 (Pin_6)
- net NRST: now also U12.7 (NRST)
- net SPI1_CS: now also U12.20 (PA4)
- net SPI1_MISO: now also U12.22 (PA6)
- net SPI1_MOSI: now also U12.23 (PA7)
- net SPI1_SCK: now also U12.21 (PA5)
- net SPI3_CS: now also U12.10 (PC2)
- net SPI3_MISO: now also U12.52 (PC11)
- net SPI3_MOSI: now also U12.9 (PC1)
- net SPI3_SCK: now also U12.51 (PC10)
- net SWCLK: now also U12.49 (PA14)
- net SWDIO: now also U12.46 (PA13)
- net USART1_RX: now also U12.43 (PA10)
- net USART1_TX: now also U12.42 (PA9)
- net at C14.1: now also U12.30 (VCAP)
- net at C15.1: now also U12.47 (VCAP_2)
- new net +3.3V_: J18.2 (Pin_2)
- new net ADC_BAT_: J16.8 (Pin_8), U12.27 (PB1)
- new net GND_: J18.1 (Pin_1)
- new net _MOTOR1_IN1: J16.4 (Pin_4), U12.50 (PA15)
- new net _MOTOR1_IN2: J16.3 (Pin_3), U12.55 (PB3)
- new net _MOTOR2_IN1: J15.1 (Pin_1), U12.29 (PB10)
- new net _MOTOR2_IN2: J15.2 (Pin_2), U12.17 (PA3)
- new net _MOTOR3_IN1: J16.2 (Pin_2), U12.56 (PB4)
- new net _MOTOR3_IN2: J16.1 (Pin_1), U12.57 (PB5)
- new net _MOTOR4_IN1: J16.9 (Pin_9), U12.26 (PB0)
- new net _MOTOR4_IN2: J16.5 (Pin_5), U12.40 (PC9)
- new net _MOTOR5_IN1: J15.8 (Pin_8), U12.58 (PB6)
- new net _MOTOR5_IN2: J15.7 (Pin_7), U12.59 (PB7)
- new net _MOTOR6_IN1: J15.6 (Pin_6), U12.61 (PB8)
- new net _MOTOR6_IN2: J15.5 (Pin_5), U12.62 (PB9)
- new net _MOTOR7_IN1: J15.4 (Pin_4), U12.14 (PA0_WKUP)
- new net _MOTOR7_IN2: J15.3 (Pin_3), U12.15 (PA1)
- new net _MOTOR8_IN1: J16.7 (Pin_7), U12.37 (PC6)
- new net _MOTOR8_IN2: J16.6 (Pin_6), U12.38 (PC7)
