File: mpu9250.kicad_sch (KiCad schematic)
At the start: 4 parts

Commit message: 回路設計済
Parts:
- C1, C2, C3: renamed from C?; footprint (none) -> Capacitor_SMD:C_0603_1608Metric_Pad1.08x0.95mm_HandSolder
- U9: renamed from U?; footprint (none) -> Package_DFN_QFN:QFN-24-1EP_3x3mm_P0.4mm_EP1.75x1.6mm
Changed lines of the file:
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@@
   (symbol (lib_id "power:GND") (at 138.43 110.49 0) (unit 1)
     (in_bom yes) (on_board yes)
-    (property "Reference" "#PWR?" (id 0) (at 138.43 116.84 0)
+    (property "Reference" "#PWR043" (id 0) (at 138.43 116.84 0)
       (effects (font (size 1.27 1.27)) hide)
     )
@@
   (symbol (lib_id "power:GND") (at 168.91 102.87 0) (unit 1)
     (in_bom yes) (on_board yes) (fields_autoplaced)
-    (property "Reference" "#PWR?" (id 0) (at 168.91 109.22 0)
+    (property "Reference" "#PWR047" (id 0) (at 168.91 109.22 0)
       (effects (font (size 1.27 1.27)) hide)
     )
@@
   (symbol (lib_id "Device:C_Small") (at 168.91 99.06 0) (unit 1)
     (in_bom yes) (on_board yes) (fields_autoplaced)
-    (property "Reference" "C?" (id 0) (at 171.45 97.7962 0)
+    (property "Reference" "C3" (id 0) (at 171.45 97.7962 0)
       (effects (font (size 1.27 1.27)) (justify left))
     )
@@
       (effects (font (size 1.27 1.27)) (justify left))
     )
-    (property "Footprint" "" (id 2) (at 168.91 99.06 0)
+    (property "Footprint" "Capacitor_SMD:C_0603_1608Metric_Pad1.08x0.95mm_HandSolder" (id 2) (at 168.91 99.06 0)
       (effects (font (size 1.27 1.27)) hide)
     )
@@
   (symbol (lib_id "power:+3.3V") (at 168.91 93.98 0) (unit 1)
     (in_bom yes) (on_board yes) (fields_autoplaced)
-    (property "Reference" "#PWR?" (id 0) (at 168.91 97.79 0)
+    (property "Reference" "#PWR046" (id 0) (at 168.91 97.79 0)
       (effects (font (size 1.27 1.27)) hide)
     )
@@
   (symbol (lib_id "power:GND") (at 162.56 83.82 0) (unit 1)
     (in_bom yes) (on_board yes) (fields_autoplaced)
-    (property "Reference" "#PWR?" (id 0) (at 162.56 90.17 0)
+    (property "Reference" "#PWR045" (id 0) (at 162.56 90.17 0)
       (effects (font (size 1.27 1.27)) hide)
     )
@@
   (symbol (lib_id "power:+3.3V") (at 110.49 101.6 0) (unit 1)
     (in_bom yes) (on_board yes) (fields_autoplaced)
-    (property "Reference" "#PWR?" (id 0) (at 110.49 105.41 0)
+    (property "Reference" "#PWR041" (id 0) (at 110.49 105.41 0)
       (effects (font (size 1.27 1.27)) hide)
     )
@@
   (symbol (lib_id "Device:C_Small") (at 114.3 106.68 0) (unit 1)
     (in_bom yes) (on_board yes)
-    (property "Reference" "C?" (id 0) (at 109.22 105.41 0)
+    (property "Reference" "C1" (id 0) (at 109.22 105.41 0)
       (effects (font (size 1.27 1.27)) (justify left))
     )
@@
       (effects (font (size 1.27 1.27)) (justify left))
     )
-    (property "Footprint" "" (id 2) (at 114.3 106.68 0)
+    (property "Footprint" "Capacitor_SMD:C_0603_1608Metric_Pad1.08x0.95mm_HandSolder" (id 2) (at 114.3 106.68 0)
       (effects (font (size 1.27 1.27)) hide)
     )
@@
   (symbol (lib_id "My_Device:MPU9250") (at 137.16 71.12 0) (unit 1)
     (in_bom yes) (on_board yes) (fields_autoplaced)
-    (property "Reference" "U?" (id 0) (at 156.21 74.7012 0))
+    (property "Reference" "U9" (id 0) (at 156.21 74.7012 0))
     (property "Value" "MPU9250" (id 1) (at 156.21 77.2412 0))
-    (property "Footprint" "" (id 2) (at 137.16 66.04 0)
+    (property "Footprint" "Package_DFN_QFN:QFN-24-1EP_3x3mm_P0.4mm_EP1.75x1.6mm" (id 2) (at 137.16 66.04 0)
       (effects (font (size 1.27 1.27)) hide)
     )
@@
   (symbol (lib_id "power:GND") (at 114.3 110.49 0) (unit 1)
     (in_bom yes) (on_board yes) (fields_autoplaced)
-    (property "Reference" "#PWR?" (id 0) (at 114.3 116.84 0)
+    (property "Reference" "#PWR042" (id 0) (at 114.3 116.84 0)
       (effects (font (size 1.27 1.27)) hide)
     )
@@
   (symbol (lib_id "power:GND") (at 140.97 104.14 0) (unit 1)
     (in_bom yes) (on_board yes)
-    (property "Reference" "#PWR?" (id 0) (at 140.97 110.49 0)
+    (property "Reference" "#PWR044" (id 0) (at 140.97 110.49 0)
       (effects (font (size 1.27 1.27)) hide)
     )
@@
   (symbol (lib_id "Device:C_Small") (at 138.43 106.68 0) (unit 1)
     (in_bom yes) (on_board yes)
-    (property "Reference" "C?" (id 0) (at 140.97 107.95 0)
+    (property "Reference" "C2" (id 0) (at 140.97 107.95 0)
       (effects (font (size 1.27 1.27)) (justify left))
     )
@@
       (effects (font (size 1.27 1.27)) (justify left))
     )
-    (property "Footprint" "" (id 2) (at 138.43 106.68 0)
+    (property "Footprint" "Capacitor_SMD:C_0603_1608Metric_Pad1.08x0.95mm_HandSolder" (id 2) (at 138.43 106.68 0)
       (effects (font (size 1.27 1.27)) hide)
     )

Commit message: 部品配置完了
Parts:
- renumbered U9 to U8
Changed lines of the file:
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@@
   (symbol (lib_id "power:GND") (at 138.43 110.49 0) (unit 1)
     (in_bom yes) (on_board yes)
-    (property "Reference" "#PWR043" (id 0) (at 138.43 116.84 0)
+    (property "Reference" "#PWR03" (id 0) (at 138.43 116.84 0)
       (effects (font (size 1.27 1.27)) hide)
     )
@@
   (symbol (lib_id "power:GND") (at 168.91 102.87 0) (unit 1)
     (in_bom yes) (on_board yes) (fields_autoplaced)
-    (property "Reference" "#PWR047" (id 0) (at 168.91 109.22 0)
+    (property "Reference" "#PWR07" (id 0) (at 168.91 109.22 0)
       (effects (font (size 1.27 1.27)) hide)
     )
@@
   (symbol (lib_id "power:+3.3V") (at 168.91 93.98 0) (unit 1)
     (in_bom yes) (on_board yes) (fields_autoplaced)
-    (property "Reference" "#PWR046" (id 0) (at 168.91 97.79 0)
+    (property "Reference" "#PWR06" (id 0) (at 168.91 97.79 0)
       (effects (font (size 1.27 1.27)) hide)
     )
@@
   (symbol (lib_id "power:GND") (at 162.56 83.82 0) (unit 1)
     (in_bom yes) (on_board yes) (fields_autoplaced)
-    (property "Reference" "#PWR045" (id 0) (at 162.56 90.17 0)
+    (property "Reference" "#PWR05" (id 0) (at 162.56 90.17 0)
       (effects (font (size 1.27 1.27)) hide)
     )
@@
   (symbol (lib_id "power:+3.3V") (at 110.49 101.6 0) (unit 1)
     (in_bom yes) (on_board yes) (fields_autoplaced)
-    (property "Reference" "#PWR041" (id 0) (at 110.49 105.41 0)
+    (property "Reference" "#PWR01" (id 0) (at 110.49 105.41 0)
       (effects (font (size 1.27 1.27)) hide)
     )
@@
   (symbol (lib_id "My_Device:MPU9250") (at 137.16 71.12 0) (unit 1)
     (in_bom yes) (on_board yes) (fields_autoplaced)
-    (property "Reference" "U9" (id 0) (at 156.21 74.7012 0))
+    (property "Reference" "U8" (id 0) (at 156.21 74.7012 0))
     (property "Value" "MPU9250" (id 1) (at 156.21 77.2412 0))
     (property "Footprint" "Package_DFN_QFN:QFN-24-1EP_3x3mm_P0.4mm_EP1.75x1.6mm" (id 2) (at 137.16 66.04 0)
@@
   (symbol (lib_id "power:GND") (at 114.3 110.49 0) (unit 1)
     (in_bom yes) (on_board yes) (fields_autoplaced)
-    (property "Reference" "#PWR042" (id 0) (at 114.3 116.84 0)
+    (property "Reference" "#PWR02" (id 0) (at 114.3 116.84 0)
       (effects (font (size 1.27 1.27)) hide)
     )
@@
   (symbol (lib_id "power:GND") (at 140.97 104.14 0) (unit 1)
     (in_bom yes) (on_board yes)
-    (property "Reference" "#PWR044" (id 0) (at 140.97 110.49 0)
+    (property "Reference" "#PWR04" (id 0) (at 140.97 110.49 0)
       (effects (font (size 1.27 1.27)) hide)
     )
